File: design/ecad/fmt.sch (KiCad schematic (older format))
At the start: 6 parts

Commit message: Added 1uF caps to switches wich makes for a better user experience.
Parts:
- added C1, C2: 1uF, symbol Device:C_Small
- gave numbers to parts that had none: 4
Connections:
- wire segments 28 -> 34
Changed lines of the file:
@@
 EESchema Schematic File Version 4
+LIBS:fmt-cache
 EELAYER 26 0
 EELAYER END
@@
 	3550 2750 3550 2800
 $Comp
-L moran:oled_128x64 U?
+L moran:oled_128x64 U1
 U 1 1 615092FC
 P 7100 4300
-F 0 "U?" H 7100 4850 50  0000 L CNN
+F 0 "U1" H 7100 4850 50  0000 L CNN
 F 1 "oled_128x64" H 6900 4650 50  0000 L CNN
 F 2 "" H 7250 4050 50  0001 C CNN
@@
 	5650 4150 5650 4900
 $Comp
-L power:GND #PWR?
+L power:GND #PWR0101
 U 1 1 61509454
 P 5650 4900
-F 0 "#PWR?" H 5650 4650 50  0001 C CNN
+F 0 "#PWR0101" H 5650 4650 50  0001 C CNN
 F 1 "GND" H 5655 4727 50  0000 C CNN
 F 2 "" H 5650 4900 50  0001 C CNN
@@
 $EndComp
 $Comp
-L power:+5V #PWR?
+L power:+5V #PWR0102
 U 1 1 61509465
 P 5900 4900
-F 0 "#PWR?" H 5900 4750 50  0001 C CNN
+F 0 "#PWR0102" H 5900 4750 50  0001 C CNN
 F 1 "+5V" H 5915 5073 50  0000 C CNN
 F 2 "" H 5900 4900 50  0001 C CNN
@@
 	6450 4350 6700 4350
 $Comp
-L moran:AS5600 U?
+L moran:AS5600 U2
 U 1 1 61509B69
 P 7150 2850
-F 0 "U?" H 7125 3715 50  0000 C CNN
+F 0 "U2" H 7125 3715 50  0000 C CNN
 F 1 "AS5600" H 7125 3624 50  0000 C CNN
 F 2 "" H 5950 3750 50  0001 C CNN
@@
 	2500 3900 2850 3900
 $Comp
-L Switch:SW_Push SW?
+L Switch:SW_Push SW2
 U 1 1 6150AAA3
-P 6950 5500
-F 0 "SW?" H 6950 5785 50  0000 C CNN
-F 1 "SW_UNIT" H 6950 5694 50  0000 C CNN
-F 2 "" H 6950 5700 50  0001 C CNN
-F 3 "" H 6950 5700 50  0001 C CNN
-	1    6950 5500
-	1    0    0    -1
-$EndComp
-$Comp
-L power:GND #PWR?
+P 7550 5050
+F 0 "SW2" H 7550 5335 50  0000 C CNN
+F 1 "SW_UNIT" H 7550 5244 50  0000 C CNN
+F 2 "" H 7550 5250 50  0001 C CNN
+F 3 "" H 7550 5250 50  0001 C CNN
+	1    7550 5050
+	1    0    0    -1
+$EndComp
+$Comp
+L power:GND #PWR0103
 U 1 1 6150ABA7
-P 7800 5600
-F 0 "#PWR?" H 7800 5350 50  0001 C CNN
-F 1 "GND" H 7805 5427 50  0000 C CNN
-F 2 "" H 7800 5600 50  0001 C CNN
-F 3 "" H 7800 5600 50  0001 C CNN
-	1    7800 5600
-	1    0    0    -1
-$EndComp
-Wire Wire Line
-	7150 5500 7800 5500
-Wire Wire Line
-	7800 5500 7800 5600
-Text GLabel 6300 5500 0    50   Input ~ 0
+P 8400 5150
+F 0 "#PWR0103" H 8400 4900 50  0001 C CNN
+F 1 "GND" H 8405 4977 50  0000 C CNN
+F 2 "" H 8400 5150 50  0001 C CNN
+F 3 "" H 8400 5150 50  0001 C CNN
+	1    8400 5150
+	1    0    0    -1
+$EndComp
+Wire Wire Line
+	7750 5050 8400 5050
+Wire Wire Line
+	8400 5050 8400 5150
+Text GLabel 6900 5050 0    50   Input ~ 0
 SW_UNIT
 Wire Wire Line
-	6750 5500 6300 5500
-$Comp
-L Switch:SW_Push SW?
+	7350 5050 7200 5050
+$Comp
+L Switch:SW_Push SW1
 U 1 1 6150B6AA
-P 6950 6000
-F 0 "SW?" H 6950 6285 50  0000 C CNN
-F 1 "SW_RESET" H 6950 6194 50  0000 C CNN
-F 2 "" H 6950 6200 50  0001 C CNN
-F 3 "" H 6950 6200 50  0001 C CNN
-	1    6950 6000
-	1    0    0    -1
-$EndComp
-$Comp
-L power:GND #PWR?
+P 7500 5700
+F 0 "SW1" H 7500 5985 50  0000 C CNN
+F 1 "SW_RESET" H 7500 5894 50  0000 C CNN
+F 2 "" H 7500 5900 50  0001 C CNN
+F 3 "" H 7500 5900 50  0001 C CNN
+	1    7500 5700
+	1    0    0    -1
+$EndComp
+$Comp
+L power:GND #PWR0104
 U 1 1 6150B6B1
-P 7800 6100
-F 0 "#PWR?" H 7800 5850 50  0001 C CNN
-F 1 "GND" H 7805 5927 50  0000 C CNN
-F 2 "" H 7800 6100 50  0001 C CNN
-F 3 "" H 7800 6100 50  0001 C CNN
-	1    7800 6100
-	1    0    0    -1
-$EndComp
-Wire Wire Line
-	7150 6000 7800 6000
-Wire Wire Line
-	7800 6000 7800 6100
-Text GLabel 6300 6000 0    50   Input ~ 0
+P 8350 5800
+F 0 "#PWR0104" H 8350 5550 50  0001 C CNN
+F 1 "GND" H 8355 5627 50  0000 C CNN
+F 2 "" H 8350 5800 50  0001 C CNN
+F 3 "" H 8350 5800 50  0001 C CNN
+	1    8350 5800
+	1    0    0    -1
+$EndComp
+Wire Wire Line
+	7700 5700 8350 5700
+Wire Wire Line
+	8350 5700 8350 5800
+Text GLabel 6850 5700 0    50   Input ~ 0
 SW_RESET
 Wire Wire Line
-	6750 6000 6300 6000
+	7300 5700 7200 5700
 Text Notes 5550 6400 0    50   ~ 0
 Note: This is the reset to zero button. It does not reset the micro-controller
+$Comp
+L Device:C_Small C1
+U 1 1 6158C265
+P 7200 5200
+F 0 "C1" H 7292 5246 50  0000 L CNN
+F 1 "1uF" H 7292 5155 50  0000 L CNN
+F 2 "" H 7200 5200 50  0001 C CNN
+F 3 "~" H 7200 5200 50  0001 C CNN
+	1    7200 5200
+	1    0    0    -1
+$EndComp
+Wire Wire Line
+	7200 5100 7200 5050
+Connection ~ 7200 5050
+Wire Wire Line
+	7200 5050 6900 5050
+$Comp
+L power:GND #PWR0105
+U 1 1 6158C626
+P 7200 5350
+F 0 "#PWR0105" H 7200 5100 50  0001 C CNN
+F 1 "GND" H 7205 5177 50  0000 C CNN
+F 2 "" H 7200 5350 50  0001 C CNN
+F 3 "" H 7200 5350 50  0001 C CNN
+	1    7200 5350
+	1    0    0    -1
+$EndComp
+Wire Wire Line
+	7200 5350 7200 5300
+$Comp
+L Device:C_Small C2
+U 1 1 6158C9B8
+P 7200 5850
+F 0 "C2" H 7292 5896 50  0000 L CNN
+F 1 "1uF" H 7292 5805 50  0000 L CNN
+F 2 "" H 7200 5850 50  0001 C CNN
+F 3 "~" H 7200 5850 50  0001 C CNN
+	1    7200 5850
+	1    0    0    -1
+$EndComp
+$Comp
+L power:GND #PWR0106
+U 1 1 6158CE02
+P 7200 6000
+F 0 "#PWR0106" H 7200 5750 50  0001 C CNN
+F 1 "GND" H 7205 5827 50  0000 C CNN
+F 2 "" H 7200 6000 50  0001 C CNN
+F 3 "" H 7200 6000 50  0001 C CNN
+	1    7200 6000
+	1    0    0    -1
+$EndComp
+Wire Wire Line
+	7200 5750 7200 5700
+Connection ~ 7200 5700
+Wire Wire Line
+	7200 5700 6850 5700
+Wire Wire Line
+	7200 6000 7200 5950
 $EndSCHEMATC
